File: kicad/trivial-lm399.sch (KiCad schematic (older format))
At the start: 14 parts, among them CON1 BARREL_JACK, P1 CONN_1, P2 CONN_1, P3 CONN_2, P4 CONN_2, P5 CONN_2, U1 OP07, U2 LM399

Commit message: rolling back to version which matches boards
Parts:
- added R1, R2, R3: ?, symbol R_0W25_1PCT
- added R7, R8: 100k, symbol R_0W25
- added RV1: ?, symbol POT
- added U3: TL062, ~, symbol TL062
- C1: value 0.1uF -> 10nF
- C2: value 0.1uF -> C_CER
- U1: value OP07 -> LM741
Connections:
- net labels added: OP_OUT, TRIM1, TRIM2
- wire segments 47 -> 90
- no-connect marks 2 -> 0
Other:
- note added: "Optional dual opamp footprint"
- note added: "Terminated opamp"
